File: Hardware/SCRB-Payload_Extension_ERC.kicad_pcb (KiCad board)
At the start: 4 copper layers, 79.3 x 57.3 mm, 107 parts, among them IC1 STM32C542CCT6, J1 Conn_UART, J11 Conn_5V, J2 Conn_LoadCell, J4 Conn_LoadCell, J5 Conn_LoadCell, J6 Conn_LoadCell, J7 Conn_Therm, J8 ST-Link-Conn-SM, J9 Conn_6HIGH, Q1 NMOS, SW1 SW_Oval, U1 TPS543x21, U2 TPD4E05U06DQAR, U3 THVD1500DR, U4 ADS1220IPW, U5 ADS1220IPW, U6 TLV75533PDBV, U7 INA241A4IDDFR, U8 TPD4E05U06DQAR, Y1 16M, 9p

Commit message: most of the layout done, awaiting if buck converter needed
Parts:
- added TP2: Testpoint, TestPoint:TestPoint_Loop_D2.60mm_Drill1.6mm_Beaded, F.Cu at (149.3, 107.0)
- added TP3: Testpoint, TestPoint:TestPoint_Loop_D2.60mm_Drill1.6mm_Beaded, F.Cu at (144.7, 70.2)
- moved U2 15.6 mm to (120.0, 117.5), turned to -90 degrees
- moved R33 14.1 mm to (131.0, 80.4), turned to 90 degrees
- moved C2 14.0 mm to (152.1, 78.7)
- moved R10 13.8 mm to (161.9, 89.4), turned to -90 degrees
- moved R35 13.2 mm to (130.1, 80.4), turned to 90 degrees
- moved R9 12.5 mm to (159.7, 89.4), turned to -90 degrees
- moved C26 12.5 mm to (162.9, 91.4), turned to 0 degrees
- moved R34 11.0 mm to (135.4, 87.3), turned to 180 degrees
- moved C25 10.9 mm to (161.1, 91.4), turned to 0 degrees
- moved R11 10.8 mm to (162.0, 103.3), turned to 90 degrees
- moved R43 10.8 mm to (163.7, 94.4), turned to 90 degrees
- moved TP1 10.5 mm to (144.7, 65.2)
- moved C31 10.1 mm to (162.9, 101.8), turned to 180 degrees
- moved C12 9.75 mm to (163.7, 96.5), turned to -90 degrees
- moved C24 9.68 mm to (159.2, 91.4), turned to 0 degrees
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Connections:
- IC1 pad 13: Net-(IC1-PA3) -> unconnected-(IC1-PA3-Pad13)
- IC1 pad 14: Net-(IC1-PA4) -> unconnected-(IC1-PA4-Pad14)
- IC1 pad 15: Net-(IC1-PA5) -> unconnected-(IC1-PA5-Pad15)
- IC1 pad 28: unconnected-(IC1-PB15-Pad28) -> Net-(IC1-PB15)
- IC1 pad 38: unconnected-(IC1-PA15-Pad38) -> Net-(IC1-PA15)
- IC1 pad 39: unconnected-(IC1-PB3-Pad39) -> Net-(IC1-PB3)
- J2 pad 3: /Sig1+ -> /Sig2+
- J2 pad 4: /Sig1- -> /Sig2-
- J4 pad 3: /Sig2+ -> /Sig1+
- J4 pad 4: /Sig2- -> /Sig1-
- Q1 pad 3: /6_Hi -> /1V5
- R30 pad 2: 6_Lo -> GND
- R33 pad 1: Net-(IC1-PA3) -> Net-(IC1-PA15)
- R34 pad 2: Net-(IC1-PA4) -> Net-(IC1-PB15)
- R35 pad 1: Net-(IC1-PA5) -> Net-(IC1-PB3)
- U7 pad 1: 6_Lo -> GND
Routing:
- net /E1-: track 0.00 -> 77.2 mm
- net Net-(IC1-PA7): track 0.00 -> 44.2 mm, vias 0 -> 2
- net /Sig2-: track 0.00 -> 43.8 mm
- net /Sig2+: track 0.00 -> 42.6 mm
- net /CURR_VOUT: track 0.00 -> 38.6 mm, vias 0 -> 2
- net /SPI2_~{CS}: track 0.00 -> 36.5 mm, vias 0 -> 2
- net Net-(IC1-PA6): track 0.00 -> 35.2 mm, vias 0 -> 2
- net /SPI2_MOSI: track 0.00 -> 31.1 mm, vias 0 -> 2
- net /E3-: track 0.00 -> 30.4 mm
- net /SPI2_SCK: track 0.00 -> 30.4 mm, vias 0 -> 2
- net /UART_TX: track 1.95 -> 29.6 mm, vias 0 -> 2
- net /UART_RX: track 0.00 -> 26.3 mm, vias 0 -> 2
- net Net-(Q1-G): track 0.00 -> 24.3 mm
- net /SPI1_MOSI: track 0.00 -> 23.3 mm, vias 0 -> 2
- net /SPI1_SCK: track 0.00 -> 21.2 mm, vias 0 -> 2
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- added copper zone on B.Cu, net /6_Hi
- added copper zone on In2.Cu, net /6_Hi
- added copper zone on B.Cu, net GND
- removed copper zone on F.Cu, net /6_Hi
- removed copper zone on In1.Cu, net /6_Hi
Other:
- board text added: "5V"
- board text added: "ST-Link"
- board text added: "UART"
- board text added: "ʕっ•ᴥ•ʔっ"
