File: Hardware/SCRB-Payload_Extension_ERC.kicad_sch (KiCad schematic)
At the start: 84 parts, among them J1 Conn_01x03, J2 Conn_LoadCell, J3 ST_Link_Conn, J4 Conn_LoadCell, J5 Conn_LoadCell, J6 Conn_01x01, J7 Conn_Therm, Q1 NMOS, SW1 SW_Tiny, U1 STM32F412RET6, U2 TPD4E05U06DQAR, U3 THVD1500DR, U4 ADS1220IPW, U5 ADS1220IPW, U6 ADS1220IPW, U7 INA241A4IDDFR, U8 TPD4E05U06DQAR, Y1 16M, 9p

Commit message: Updated ERC board schematic
Parts:
- removed C18, C23: 0.1uF, SCRB_STD_Passives:C0402, symbol SCRB_STD_Passives:C0402
- removed C22: 5.1nF, SCRB_STD_Passives:C0402, symbol SCRB_STD_Passives:C0402
- removed J3: ST_Link_Conn, Connector_JST:JST_GH_BM04B-GHS-TBT_1x04-1MP_P1.25mm_Vertical, symbol Connector_Generic:Conn_01x04
- removed U6: ADS1220IPW, ADS1220:PW16, symbol ADS1220:ADS1220IPW
- added IC1: STM32C542CCT6, SCRB_Misc_ICs:LQFP-48_7x7mm_P0.5mm, symbol STM32C542CCT6:STM32C542CCT6
- added J10: Conn_01x01, symbol Connector_Generic:Conn_01x01
- added J11: Conn_5V, SCRB_STD_Passives:R0402, symbol Connector_Generic:Conn_01x02
- added J8: ST-Link-Conn-SM, Connector_JST:JST_PH_B4B-PH-SM4-TB_1x04-1MP_P2.00mm_Vertical, symbol SCRB_EIFs:ST-Link_Conn-4-SM
- added J9: Conn_20HIGH, Connector_AMASS:AMASS_XT30U-M_1x02_P5.0mm_Vertical, symbol Connector_Generic:Conn_01x02
- added R26, R31: 470, SCRB_STD_Passives:R0402, symbol SCRB_STD_Passives:R0402
- added TP1: Testpoint, TestPoint:TestPoint_Loop_D2.60mm_Drill1.6mm_Beaded, symbol SCRB_Connectors:TP
- C28: value 5.1nF -> 16nF
- C8: value 5.1nF -> 6.8nF
- R10, R9: value 100 -> 470
Connections:
- net 3V3: now also J8.1 (3V3)
- net 5V: now also J11.1 (Pin_1), R26.2; no longer C8.1, U4.11 (AIN0/REFP1)
- net AIN1_1: now also C11.1, C9.2, R4.2; no longer C10.2, C9.1, R3.2
- net AIN1_3: now also U5.10 (AIN1)
- net AIN2_2: now also C13.2, C15.1, R5.2, U4.7 (AIN2); no longer C15.2, C17.1, R6.2, U5.7 (AIN2)
- net AIN2_3: now also U5.7 (AIN2)
- net E1-: now also J2.2 (Pin_2), J4.2 (Pin_2), R31.2; no longer C8.2, J2.3 (Pin_3), U4.6 (AIN3/REFN1)
- net E3-: now also J5.2 (Pin_2), U5.6 (AIN3/REFN1); no longer J5.3 (Pin_3)
- net GND: now also J11.2 (Pin_2), J8.4 (GND); no longer R30.2, U7.1 (IN-)
- net Nichrome_wire: no longer J6.1 (Pin_1)
- net SYS_SWDCLK: now also J8.3 (SWCLK)
- net SYS_SWDIO: now also J8.2 (SWDIO)
- net Sig1+: now also J2.3 (Pin_3); no longer J2.2 (Pin_2)
- net Sig2+: now also J4.3 (Pin_3); no longer J4.2 (Pin_2)
- net Sig3+: now also J5.3 (Pin_3); no longer J5.2 (Pin_2)
- net at Q1.1 (G), R27.1, R28.2: now also TP1.1
- net REFN0: now reaches U4.8 (REFN0)
- net REFN0: now also C8.2, R31.1
- net REFP0: now reaches U4.9 (REFP0)
- net REFP0: now also C8.1, R26.1
- removed net AIN1_2: C13.2, C15.1, R5.2, U5.10 (AIN1)
- removed net AIN2_1: C11.1, C9.2, R4.2, U4.7 (AIN2)
- removed net E2-: J4.3 (Pin_3), U5.6 (AIN3/REFN1)
- new net 20_Hi: J6.1 (Pin_1), J9.1 (Pin_1)
- new net 20_Lo: J10.1 (Pin_1), J9.2 (Pin_2), R30.2, U7.1 (IN-)
- new net AIN0_1: C10.2, C9.1, R3.2, U4.11 (AIN0/REFP1)
- new net AIN3_2: C15.2, C17.1, R6.2, U4.6 (AIN3/REFN1)
- no-connect marks 43 -> 38
Other:
- note added: "FIND APPROPRIATE RESISTOR + optocoupler"
- note added: "First order differential, common-mode RC filter: f_cMAX = f_MOD/10 = 256kHz/10 = 25.6kHz Load cell specs: R_in = 405 | R_out = 350 | Excitation = 5V R_F1 <= 1k -> R_F1,2 = 470 C_DIF1 = 1/(2π * (350+470+470) * 25.6kHz) = 4.82nF -> 5.1nF C_CM1,2 = C_DIF1/10 = 510Pf f_diff = 1/(2π * (350+470+470) * C_DIF1) = 24.2kHz C_DIF2 = 1/(2π * 405 * 24.2kHz) = 16.24nF -> 16nF f_ref = 1/(2π * 405 * 16nF) = 24.6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"
- note removed: "FIND APPROPRIATE RESISTOR"

Commit message: added extra load cell on schematic
Parts:
- removed C14, C4, C5, C6: 0.1uF, SCRB_STD_Passives:C0402, symbol SCRB_STD_Passives:C0402
- removed C19, C3: 4.7uF, SCRB_STD_Passives:C0603, symbol SCRB_STD_Passives:C0603
- removed C28: 16nF, SCRB_STD_Passives:C0402, symbol SCRB_STD_Passives:C0402
- removed J10, J6: Conn_01x01, symbol Connector_Generic:Conn_01x01
- removed R13, R14, R15, R16, R17, R18, R19, R20, R21, R22, R23: 47, SCRB_STD_Passives:R0402, symbol SCRB_STD_Passives:R0402
- removed R24, R25: 4.7k, SCRB_STD_Passives:R0402, symbol SCRB_STD_Passives:R0402
- removed SW1: SW_Tiny, SCRB_Electromechanical:SW_C913791, symbol SCRB_Electromechanical:SW_Tiny
- removed U1: STM32F412RET6, Package_QFP:LQFP-64_10x10mm_P0.5mm, symbol MCU_ST_STM32F4:STM32F412RETx
- added C18: 1uF, SCRB_STD_Passives:C0402, symbol SCRB_STD_Passives:C0402
- added C22, C23, C32, C36: 0.1uF, SCRB_STD_Passives:C0402, symbol SCRB_STD_Passives:C0402
- added C33: 0.1unF, SCRB_STD_Passives:C0402, symbol SCRB_STD_Passives:C0402
- added C34: 4.7uF, SCRB_STD_Passives:C0402, symbol SCRB_STD_Passives:C0402
- added C35: 2.2uF, SCRB_STD_Passives:C0603, symbol SCRB_STD_Passives:C0603
- added C37: 10nF, SCRB_STD_Passives:C0402, symbol SCRB_STD_Passives:C0402
- added C38: 5.1nF, SCRB_STD_Passives:C0402, symbol SCRB_STD_Passives:C0402
- added C39: 510pF, SCRB_STD_Passives:C0402, symbol SCRB_STD_Passives:C0402
- added IC2: AOZ2260AQI-15, AOZ2260AQI15, symbol AOZ2260AQI-15:AOZ2260AQI-15
- added J6: Conn_LoadCell, Connector_JST:JST_XH_B4B-XH-A_1x04_P2.50mm_Vertical, symbol Connector_Generic:Conn_01x04
- added LD3: LED0603, SCRB_STD_Actives:LED0603, symbol SCRB_STD_Actives:LED0603
- added R32: 10k, SCRB_STD_Passives:R0402, symbol SCRB_STD_Passives:R0402
- added R33, R34, R35, R36, R37, R38, R39, R40: 47, SCRB_STD_Passives:R0402, symbol SCRB_STD_Passives:R0402
- added R41, R42: 4.7K, SCRB_STD_Passives:R0402, symbol SCRB_STD_Passives:R0402
- added R43, R44: 470, SCRB_STD_Passives:R0402, symbol SCRB_STD_Passives:R0402
- added SW1: SW_Oval, SCRB_Electromechanical:SW_C2888430, symbol SCRB_Electromechanical:SW_Oval
- added U6: TLV75533PDBV, Package_TO_SOT_SMD:SOT-23-5, symbol Regulator_Linear:TLV75533PDBV
- C12: value 0.1uF -> 6.8nF; Voltage 10V -> 25V
- C31: value 10nF -> 510pF; Voltage Voltage -> 25V
- R11: value 10k -> 470
- R12: value 47 -> 470
- R29: value 270 -> 680
Connections:
- net Nichrome_wire is gone; now on net 20_Hi: Q1.3 (D)
- net 3V3: now also IC1.24 (VDD_1), IC1.36 (VDD_2), IC1.48 (VDD_3), C22.1, C23.2, C32.2, C33.2, C34.2, R32.1, U6.5 (OUT); no longer C12.1
- net 5V: now also C18.1, J6.1 (Pin_1), R41.1, R42.1, R43.2, U6.1 (IN), U6.3 (EN); no longer U5.11 (AIN0/REFP1)
- net ADC_Therm: now also IC1.11 (PA1), C37.1; no longer C31.1
- net AIN1_3: now also C25.2, C26.1, R10.2; no longer C24.2, C25.1, R9.2
- net CURR_VOUT: now also IC1.12 (PA2)
- net E3-: now also J6.2 (Pin_2), R44.2; no longer U5.6 (AIN3/REFN1)
- net GATE_SW: now also IC1.29 (PA8)
- net GND: now also C31.1, IC1.23 (VSS_1), IC1.35 (VSS_2), IC1.47 (VSS_3), IC1.8 (VREF-), C18.2, C22.2, C23.1, C32.1, C33.1, C34.1, C35.2, C36.2, C37.2, C39.2, LD3.1 (K), SW1.1, U6.2 (GND); no longer C12.2, C31.2, R11.1, R12.1
- net LED_PANIK: now also IC1.2 (PC13)
- net LED_RUN: now also IC1.1 (PE2)
- net NRST: now also IC1.7 (NRST), SW1.2
- net RCC_OSC_IN: now also IC1.5 (PH0-OSC_IN)
- net RCC_OSC_OUT: now also IC1.6 (PH1-OSC_OUT)
- net SPI1_MISO: now also R36.2; no longer R12.2
- net SPI1_MOSI: now also R34.1
- net SPI1_SCK: now also R35.2
- net SPI1_~{CS}: now also R33.2
- net SPI2_MISO: now also R37.2
- net SPI2_MOSI: now also R39.2
- net SPI2_SCK: now also R40.2
- net SPI2_~{CS}: now also R38.2
- net SYS_SWDCLK: now also IC1.37 (PA14)
- net SYS_SWDIO: now also IC1.34 (PA13)
- net UART_RX: now also IC1.25 (PB12), R42.2
- net UART_TX: now also IC1.26 (PB13), R41.2
- net AIN2_4: now reaches R11.2
- net AIN2_4: now also C31.2, U5.7 (AIN2), C38.1
- net REFN0_2: now reaches U5.8 (REFN0)
- net REFN0_2: now also C12.2, R44.1
- net REFP0_2: now reaches U5.9 (REFP0)
- net REFP0_2: now also C12.1, R43.1
- net at IC1.13 (PA3): now also R33.1
- net at IC1.14 (PA4): now also R34.2
- net at IC1.15 (PA5): now also R35.1
- net at IC1.16 (PA6): now also R36.1
- net at IC1.17 (PA7): now also R37.1
- net at IC1.19 (PB1): now also R38.1
- net at IC1.20 (PB2): now also R39.1
- net at IC1.21 (PB10): now also R40.1
- net at IC1.22 (VCAP): now also C35.1
- net at IC1.9 (VREF+): now also C36.1
- removed net AIN2_3: C25.2, C26.1, R10.2, U5.7 (AIN2)
- new net: LD3.2 (A), R32.2
- new net AIN0_3: C24.2, C25.1, R9.2, U5.11 (AIN0/REFP1)
- new net AIN3_4: C38.2, C39.1, R12.2, U5.6 (AIN3/REFN1)
- new net Sig4+: J6.3 (Pin_3)
- new net Sig4-: J6.4 (Pin_4)
- no-connect marks 38 -> 27
Other:
- note added: "LDO + 20V high"
- moved on the sheet: C10, C11, C13, C15, C16, C17, C2, C20, C21, C24, C25, C26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

Commit message: working on buck converter wiring
Parts:
- removed IC2: AOZ2260AQI-15, AOZ2260AQI15, symbol AOZ2260AQI-15:AOZ2260AQI-15
- added C14: 22nF, SCRB_STD_Passives:C0402, symbol SCRB_STD_Passives:C0402
- added C19: C0402, SCRB_STD_Passives:C0402, symbol SCRB_STD_Passives:C0402
- added C3, C4, C5: 10uF, SCRB_STD_Passives:C0402, symbol SCRB_STD_Passives:C0402
- added C6: 0.1uF, SCRB_STD_Passives:C0402, symbol SCRB_STD_Passives:C0402
- added L1: L0805, SCRB_STD_Passives:L0805, symbol SCRB_STD_Passives:L0805
- added R15: R0402, SCRB_STD_Passives:R0402, symbol SCRB_STD_Passives:R0402
- added R16: 30k, SCRB_STD_Passives:R0603, symbol SCRB_STD_Passives:R0603
- added R17: 45k, SCRB_STD_Passives:R0603, symbol SCRB_STD_Passives:R0603
- added SB1: SB0402, SCRB_STD_Passives:JP0402_NO, symbol SCRB_STD_Passives:SB0402
- added U1: TPS543x21, VQFN-HR9_RQF_TEX, symbol TPS54x38:TPS54438RQFR
- C33: value 0.1unF -> 0.1uF
- J11: footprint SCRB_STD_Passives:R0402 -> Connector_JST:JST_XH_B2B-XH-AM_1x02_P2.50mm_Vertical
Connections:
- net 20_Hi: now also C14.1, C3.1, C4.1, C5.1, C6.1, U1.5 (VIN), U1.6 (VIN)
- net 20_Lo: now also C14.2, C3.2, C4.2, C5.2, C6.2, R15.2, R16.2
- new net: R16.1, R17.2, U1.3 (FB)
- new net: R15.1, U1.7 (MODE)
- new net: L1.1, U1.8 (SW)
Other:
- note added: "LDO"
- note added: "RFBT = RFBB * (Vout - Vref)/Vref = 30k * (1.5V - 0.6V)/0.6V = 45k"
- note removed: "LDO + 20V high"
- moved on the sheet: J9

Commit message: PCB layout in progress
Parts:
- removed C19: C0402, SCRB_STD_Passives:C0402, symbol SCRB_STD_Passives:C0402
- removed C34: 4.7uF, SCRB_STD_Passives:C0402, symbol SCRB_STD_Passives:C0402
- removed C4: 10uF, SCRB_STD_Passives:C0402, symbol SCRB_STD_Passives:C0402
- removed C6: 0.1uF, SCRB_STD_Passives:C0402, symbol SCRB_STD_Passives:C0402
- added C4: 68u, SCRB_STD_Passives:C0603, symbol SCRB_STD_Passives:C0603
- added C6: 4.7u, SCRB_STD_Passives:C0603, symbol SCRB_STD_Passives:C0603
- added D1: D_Zener, Diode_THT:D_DO-41_SOD81_P10.16mm_Horizontal, symbol Device:D_Zener
- added D2: SMBJ6.0CA, SCRB_STD_Actives:SMB, symbol SCRB_STD_Actives:TVS_SMB
- added R13: 121k, SCRB_STD_Passives:R0402, symbol SCRB_STD_Passives:R0402
- added R14: 54.9k, SCRB_STD_Passives:R0402, symbol SCRB_STD_Passives:R0402
- added R18: 100k, SCRB_STD_Passives:R0402, symbol SCRB_STD_Passives:R0402
- added R19: R0402, SCRB_STD_Passives:R0402, symbol SCRB_STD_Passives:R0402
- added TP2, TP3: Testpoint, TestPoint:TestPoint_Loop_D2.60mm_Drill1.6mm_Beaded, symbol SCRB_Connectors:TP
- C14: value 22nF -> 0.1u
- C3: value 10uF -> 10u
- C5: value 10uF -> 20p; Voltage 35V -> 16V
- H1, H2, H3, H4: footprint MountingHole:MountingHole_3.2mm_M3_DIN965_Pad -> MountingHole:MountingHole_3.2mm_M3
- J1: value Conn_01x03 -> Conn_UART
- J2, J4, J5, J6: footprint Connector_JST:JST_XH_B4B-XH-A_1x04_P2.50mm_Vertical -> Connector_JST:JST_PH_B4B-PH-SM4-TB_1x04-1MP_P2.00mm_Vertical
- J9: value Conn_20HIGH -> Conn_6HIGH
- L1: value L0805 -> 3.7u
- LD3: value LED0603 -> 3V3_LED
- R15: value R0402 -> 18k
Connections:
- net 3V3: now also SB1.2 (B), C6.2; no longer C22.1, R32.1, U6.5 (OUT)
- net 5V: now also D2.2 (A2), R18.1; no longer J11.1 (Pin_1)
- net GND: now also C14.2, C3.2, J9.2 (Pin_2), R15.2, R16.2, U1.4 (GND), C4.2, C6.1, D1.2 (A), R14.2, R19.1
- net Sig4+: now also R11.1
- net Sig4-: now also R12.1
- net at IC1.21 (PB10), R40.1: now also TP2.1
- net at R16.1, R17.2, U1.3 (FB): now also C5.2
- net at U1.1 (RT/SYNC): now also R19.2
- net EN: now reaches U1.2 (EN)
- net EN: now also D1.1 (K), R13.2, R14.1
- net at U1.9 (SS/PG): now also R18.2
- net 1V5: now reaches L1.2
- net 1V5: now also C5.1, Q1.3 (D), R17.1, C4.1
- net at IC1.15 (PA5), R35.1: now also TP3.1
- net ldo_3V3: now reaches SB1.1 (A)
- net ldo_3V3: now also C22.1, R32.1, U6.5 (OUT)
- net 20_Hi renamed 6_Hi
- net 6_Hi: now also R13.1; no longer C5.1, Q1.3 (D)
- removed net 20_Lo: C14.2, C3.2, C5.2, J9.2 (Pin_2), R15.2, R16.2, R30.2, U7.1 (IN-)
- new net 6_Lo: R30.2, U7.1 (IN-)
- new net tvs_5V: D2.1 (A1), J11.1 (Pin_1)
Other:
- note added: "Buck Converter for Heating Element"
- note added: "First order differential, common-mode RC filter: f_cMAX = f_MOD/10 = 256kHz/10 = 25.6kHz Load cell specs: R_in = 405 | R_out = 350 | Excitation = 5V R_F1 <= 1k -> R_F1,2 = 470 C_DIF1 = 1/(2π * (350+470+470) * 25.6kHz) = 4.82nF -> 5.1nF C_CM1,2 = C_DIF1/10 = 510Pf C_DIF2 = 1/(2π * 940 * 24.2kHz) = 6.99nF -> 6.8nF f_ref = 1/(2π * 940 * 6.8nF) = 24.9kHz"
- note added: "UVLO = 3.77 V"
- note removed: "CONNECTIONS FOR POWER!!"
- note removed: "FIND APPROPRIATE RESISTOR + optocoupler"
- note removed: "FINISH NICHROME CONNECTION"
- note removed: "First order differential, common-mode RC filter: f_cMAX = f_MOD/10 = 256kHz/10 = 25.6kHz Load cell specs: R_in = 405 | R_out = 350 | Excitation = 5V R_F1 <= 1k -> R_F1,2 = 470 C_DIF1 = 1/(2π * (350+470+470) * 25.6kHz) = 4.82nF -> 5.1nF C_CM1,2 = C_DIF1/10 = 510Pf f_diff = 1/(2π * (350+470+470) * C_DIF1) = 24.2kHz C_DIF2 = 1/(2π * 405 * 24.2kHz) = 16.24nF -> 16nF f_ref = 1/(2π * 405 * 16nF) = 24.6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"
- moved on the sheet: C14, C18, C22, C3, J9, L1, LD3, R15, R16, R17, R32, SB1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

Commit message: most of the layout done, awaiting if buck converter needed
Connections:
- net 6_Lo is gone; now on net GND: R30.2, U7.1 (IN-)
- net Sig1+: now also J4.3 (Pin_3); no longer J2.3 (Pin_3)
- net Sig1-: now also J4.4 (Pin_4); no longer J2.4 (Pin_4)
- net Sig2+: now also J2.3 (Pin_3); no longer J4.3 (Pin_3)
- net Sig2-: now also J2.4 (Pin_4); no longer J4.4 (Pin_4)
- net at R35.1, TP3.1: now also IC1.39 (PB3); no longer IC1.15 (PA5)
- net at R34.2: now also IC1.28 (PB15); no longer IC1.14 (PA4)
- net at R33.1: now also IC1.38 (PA15); no longer IC1.13 (PA3)
Other:
- moved on the sheet: C23, C32, C33, C6, R33, R34, R35, TP3
